Commit message: after ssh

File: bigbot_description/urdf/bigbot3.xacro (robot description, xacro)
@@ -50,9 +50,9 @@
 	<xacro:macro name="cylinder_inertial" params="m r h">
 		<inertial>
-			 <mass value="${m}" />
+			<mass value="${m}" />
 			<inertia  ixx="${m*(3*r*r+h*h)/12}" ixy = "0" ixz = "0"
 	      		iyy="${m*(3*r*r+h*h)/12}" iyz = "0"
 	      		izz="${m*r*r/2}" />
-               </inertial>
+        </inertial>
 	</xacro:macro>
 	<!-- per https://en.wikipedia.org/wiki/List_of_moments_of_inertia
@@ -80,9 +80,9 @@
         <!-- 		<xacro:default_inertial mass="0.0001"/> error said to remove this from footprint-->
 	<link name="base_footprint">
-		<pose xyz="0 0 .001" rpy="0 0 0"
+		<pose xyz="0 0 .001" rpy="0 0 0" />
    		<visual>
 			<geometry>
       				<box size="0.001 0.001 0.001"/>
-     			</geometry>
+     		</geometry>
 			<origin rpy="0 0 0" xyz="0 0 0"/>
 			<material name="Red"/>
@@ -283,5 +283,5 @@
       <robotBaseFrame>base_footprint</robotBaseFrame>
     </plugin>
-	</gazebo>
+  </gazebo>
 <gazebo reference="laser_frame">
     <sensor type="gpu_ray" name="head_hokuyo_sensor">

File: bigbot_description/urdf/robot2.urdf (robot description, URDF)
Before this commit: robot bigbot, 7 links, 6 joints
Links:
- link left_wheel: geometry collision cylinder length=0.0435 radius=0.085; visual cylinder length=0.0435 radius=0.085
- link right_wheel: geometry collision cylinder length=0.0435 radius=0.085; visual cylinder length=0.0435 radius=0.085
