Commit message: Increased mass to 25kg

File: bigbot_description/urdf/bigbot.xacro (robot description, xacro)
@@ -24,5 +24,5 @@
 	</material>
 	<!-- Defining parameters-->
-	<xacro:property name="mass_base" value="12" />
+	<xacro:property name="mass_base" value="24" />
 	<xacro:property name="length_base" value="0.7001" /> <!-- 27 9/16-->
 	<xacro:property name="width_base" value="0.60325" /><!--23.75 -->

File: bigbot_description/urdf/bigbot2.xacro (robot description, xacro)
@@ -28,5 +28,5 @@
 	</material>
 	<!-- Defining parameters-->
-	<xacro:property name="mass_base" value="12" />
+	<xacro:property name="mass_base" value="24" />
 	<xacro:property name="length_base" value="0.7001" /> <!-- 27 9/16 in-->
 	<xacro:property name="width_base" value="0.60325" /><!--23.75 in -->

File: bigbot_description/urdf/bigbot3.xacro (robot description, xacro)
@@ -28,5 +28,5 @@
 	</material>
 	<!-- Defining parameters-->
-	<xacro:property name="mass_base" value="12" />
+	<xacro:property name="mass_base" value="24" />
 	<xacro:property name="length_base" value="0.7001" /> <!-- 27 9/16-->
 	<xacro:property name="width_base" value="0.60325" /><!--23.75 -->

File: bigbot_description/urdf/bigbot3a.xacro (robot description, xacro)
@@ -24,5 +24,5 @@
 	</material>
 	<!-- Defining parameters-->
-	<xacro:property name="mass_base" value="12" />
+	<xacro:property name="mass_base" value="24" />
 	<xacro:property name="length_base" value="0.7001" /> <!-- 27 9/16-->
 	<xacro:property name="width_base" value="0.60325" /><!--23.75 -->

File: bigbot_description/urdf/bigbot4.xacro (robot description, xacro)
@@ -29,5 +29,5 @@
 	</material>
 	<!-- Defining parameters-->
-	<xacro:property name="mass_base" value="12" />
+	<xacro:property name="mass_base" value="24" />
 	<xacro:property name="length_base" value="0.7001" /> <!-- 27 9/16-->
 	<xacro:property name="width_base" value="0.60325" /><!--23.75 -->
